Commit message: [update]

File: install/vicpinky_description/share/vicpinky_description/urdf/camera.xacro (robot description, xacro)
@@ -3,6 +3,7 @@
     <xacro:arg name="namespace" default=""/>
     <property name="prefix" value="$(arg namespace)"/>
+    <xacro:arg name="use_gazebo" default="true"/>
   <gazebo reference="${prefix}camera_link">
-    <sensor name="rgbd_camera" type="rgbd_camera">
+    <sensor name="camera" type="rgbd_camera">
       <camera>
         <horizontal_fov>1.047</horizontal_fov>
@@ -19,5 +20,5 @@
       <update_rate>30</update_rate>
       <visualize>true</visualize>
-      <topic>astra</topic>
+      <topic>depth_camera</topic>
     </sensor>
   </gazebo>

File: install/vicpinky_description/share/vicpinky_description/urdf/robot_core.xacro (robot description, xacro)
@@ -260,5 +260,5 @@
       <parent link="${prefix}camera_mount"/>
       <child link="${prefix}camera_link"/>
-      <origin xyz="0.015 0.015 0.008" rpy="0 0 0"/>
+      <origin xyz="0.035 0.015 0.008" rpy="0 0 0"/>
     </joint>
 </robot>
