Commit message: [add]

File: vicpinky_description/urdf/camera.xacro (robot description, xacro)
@@ -1,30 +1,25 @@
 <?xml version="1.0"?>
-<robot xmlns:xacro="http://www.ros.org/wiki/xacro" >
-    <gazebo reference="camera_link">
-        <sensor name="camera" type="camera">
-            <always_on>true</always_on>
-            <visualize>true</visualize>
-            <update_rate>30</update_rate>
-            <topic>camera/image_raw</topic>
-            <gz_frame_id>camera_rgb_frame</gz_frame_id>
-            <camera name="intel_realsense_r200">
-                <camera_info_topic>camera/camera_info</camera_info_topic>
-                <horizontal_fov>1.08</horizontal_fov>
-                <image>
-                    <width>1280</width>
-                    <height>720</height>
-                    <format>R8G8B8</format>
-                </image>
-                <clip>
-                    <near>0.02</near>
-                    <far>300</far>
-                </clip>
-                <noise>
-                <type>gaussian</type>
-                    <mean>0.0</mean>
-                    <stddev>0.01</stddev>
-                </noise>
-            </camera>
-        </sensor>
-    </gazebo>
+<robot xmlns:xacro="http://www.ros.org/wiki/xacro">
+    <xacro:arg name="namespace" default=""/>
+    <property name="prefix" value="$(arg namespace)"/>
+  <gazebo reference="${prefix}camera_link">
+    <sensor name="rgbd_camera" type="rgbd_camera">
+      <camera>
+        <horizontal_fov>1.047</horizontal_fov>
+        <image>
+          <width>640</width>
+          <height>480</height>
+        </image>
+        <clip>
+          <near>0.6</near>
+          <far>8.0</far>
+        </clip>
+      </camera>
+      <always_on>1</always_on>
+      <update_rate>30</update_rate>
+      <visualize>true</visualize>
+      <topic>astra</topic>
+      <gz_frame_id>${prefix}camera_link</gz_frame_id>
+    </sensor>
+  </gazebo>
 </robot>

File: vicpinky_description/urdf/robot.urdf.xacro (robot description, xacro)
@@ -7,4 +7,4 @@
     <xacro:include filename="gazebo_control.xacro"/>
     <xacro:include filename="lidar.xacro" />
-    <xacro:include filename="camera.xacro"/>
+    <xacro:include filename="camera.xacro" />
 </robot>

File: vicpinky_description/urdf/robot_core.xacro (robot description, xacro)
@@ -235,3 +235,30 @@
         <origin xyz="0.0 0 0.03" rpy="0 0 ${pi}"/>
     </joint>
+    <link name="${prefix}camera_mount">
+      <visual>
+        <geometry>
+          <mesh filename="package://vicpinky_description/meshes/visual/orbbec_astra_camera.dae"/>
+        </geometry>
+      </visual>
+      <collision>
+        <geometry>
+          <box size="0.06 0.17 0.048"/>
+        </geometry>
+      </collision>
+      <inertial>
+        <mass value="0.22" />
+        <inertia ixx="0.000513" ixy="0.0" ixz="0.0" iyy="0.000086" iyz="0.0" izz="0.0005"/>
+      </inertial>
+    </link>
+    <joint name="${prefix}camera_mount_fixed_joint" type="fixed">
+      <parent link="${prefix}base_link"/>
+      <child link="${prefix}camera_mount"/>
+      <origin xyz="0.07 0 0.56" rpy="0 0 0"/>
+    </joint>
+    <link name="${prefix}camera_link"/>
+    <joint name="${prefix}camera_link_fixed_joint" type="fixed">
+      <parent link="${prefix}camera_mount"/>
+      <child link="${prefix}camera_link"/>
+      <origin xyz="0.015 0.015 0.008" rpy="0 0 0"/>
+    </joint>
 </robot>

Commit message: [depth urdf update]

File: vicpinky_description/urdf/camera.xacro (robot description, xacro)
@@ -5,5 +5,5 @@
     <xacro:arg name="use_gazebo" default="true"/>
   <gazebo reference="${prefix}camera_link">
-    <sensor name="camera" type="rgbd_camera">
+    <sensor name="rgbd_camera" type="rgbd_camera">
       <camera>
         <horizontal_fov>1.047</horizontal_fov>
@@ -11,14 +11,17 @@
           <width>640</width>
           <height>480</height>
+          <format>R8G8B8</format>
         </image>
         <clip>
-          <near>0.6</near>
+          <near>0.2</near>
           <far>8.0</far>
         </clip>
+        <optical_frame_id>camera_link</optical_frame_id>
       </camera>
       <always_on>1</always_on>
-      <update_rate>30</update_rate>
+      <update_rate>20</update_rate>
       <visualize>true</visualize>
-      <topic>depth_camera</topic>
+      <topic>camera</topic>
+      <gz_frame_id>camera_link</gz_frame_id>
     </sensor>
   </gazebo>

File: vicpinky_description/urdf/robot_core.xacro (robot description, xacro)
@@ -235,5 +235,5 @@
         <origin xyz="0.0 0 0.03" rpy="0 0 ${pi}"/>
     </joint>
-    <link name="${prefix}camera_mount">
+    <link name="${prefix}camera_link">
       <visual>
         <geometry>
@@ -251,13 +251,14 @@
       </inertial>
     </link>
-    <joint name="${prefix}camera_mount_fixed_joint" type="fixed">
+    <joint name="${prefix}camera_joint" type="fixed">
       <parent link="${prefix}base_link"/>
-      <child link="${prefix}camera_mount"/>
+      <child link="${prefix}camera_link"/>
       <origin xyz="0.07 0 0.56" rpy="0 0 0"/>
     </joint>
-    <link name="${prefix}camera_link"/>
-    <joint name="${prefix}camera_link_fixed_joint" type="fixed">
-      <parent link="${prefix}camera_mount"/>
-      <child link="${prefix}camera_link"/>
+    <link name="camera_link_optical">
+    </link>
+    <joint name="${prefix}camera_optical_joint" type="fixed">
+      <parent link="${prefix}camera_link"/>
+      <child link="${prefix}camera_link_optical"/>
       <origin xyz="0.035 0.015 0.008" rpy="0 0 0"/>
     </joint>

Commit message: [slam] vlam 업데이트

File: vicpinky_description/urdf/camera.xacro (robot description, xacro)
@@ -17,5 +17,5 @@
           <far>8.0</far>
         </clip>
-        <optical_frame_id>camera_link</optical_frame_id>
+        <optical_frame_id>camera_link_optical</optical_frame_id>
       </camera>
       <always_on>1</always_on>

File: vicpinky_description/urdf/robot.urdf.xacro (robot description, xacro)
@@ -8,3 +8,4 @@
     <xacro:include filename="lidar.xacro" />
     <xacro:include filename="camera.xacro" />
+    <xacro:include filename="imu.xacro" />
 </robot>

File: vicpinky_description/urdf/robot_core.xacro (robot description, xacro)
@@ -188,4 +188,5 @@
         </xacro:inertial_sphere>
     </link>
+    <!-- LIDAR -->
     <link name="${prefix}lidar_mount">
         <visual>
@@ -235,4 +236,5 @@
         <origin xyz="0.0 0 0.03" rpy="0 0 ${pi}"/>
     </joint>
+    <!-- Camera -->
     <link name="${prefix}camera_link">
       <visual>
@@ -261,5 +263,13 @@
       <parent link="${prefix}camera_link"/>
       <child link="${prefix}camera_link_optical"/>
-      <origin xyz="0.035 0.015 0.008" rpy="0 0 0"/>
-    </joint>
+      <origin xyz="0.035 0.015 0.008" rpy="-1.570796 -0.0 -1.570796"/>
+    </joint>
+    <!-- IMU -->
+    <joint name="imu_joint" type="fixed">
+        <origin xyz="0 0 0" rpy="0 0 0" />
+        <parent link="base_link"/>
+        <child link="imu_link" />
+    </joint>
+    <link name="imu_link">
+    </link>
 </robot>

Commit message: [update]

File: vicpinky_description/urdf/camera.xacro (robot description, xacro)
@@ -17,5 +17,5 @@
           <far>8.0</far>
         </clip>
-        <optical_frame_id>camera_link_optical</optical_frame_id>
+        <frame_name>camera_rgb_optical_frame</frame_name>
       </camera>
       <always_on>1</always_on>

File: vicpinky_description/urdf/robot_core.xacro (robot description, xacro)
@@ -258,10 +258,13 @@
       <origin xyz="0.07 0 0.56" rpy="0 0 0"/>
     </joint>
-    <link name="camera_link_optical">
-    </link>
+    <link name="${prefix}camera_rgb_optical_frame"/>
     <joint name="${prefix}camera_optical_joint" type="fixed">
       <parent link="${prefix}camera_link"/>
-      <child link="${prefix}camera_link_optical"/>
-      <origin xyz="0.035 0.015 0.008" rpy="-1.570796 -0.0 -1.570796"/>
+      <child link="${prefix}camera_rgb_optical_frame"/>
+      <origin xyz="0.035 0.015 0.008" rpy="0 0 0"/>
+      <pose>0 0 0 -1.57079632679 0 -1.57079632679</pose>
+      <axis>
+        <xyz>0 0 1</xyz>
+      </axis>
     </joint>
     <!-- IMU -->

Commit message: [rtabmap update]

File: vicpinky_description/urdf/camera.xacro (robot description, xacro)
@@ -1,9 +1,15 @@
 <?xml version="1.0"?>
 <robot xmlns:xacro="http://www.ros.org/wiki/xacro">
-    <xacro:arg name="namespace" default=""/>
-    <property name="prefix" value="$(arg namespace)"/>
-    <xacro:arg name="use_gazebo" default="true"/>
+  <xacro:arg name="namespace" default=""/>
+  <property name="prefix" value="$(arg namespace)"/>
+  <xacro:arg name="use_gazebo" default="true"/>
+  <link name="${prefix}camera_rgb_optical_frame"></link>
+  <joint name="${prefix}camera_optical_joint" type="fixed">
+    <parent link="${prefix}camera_link"/>
+    <child link="${prefix}camera_rgb_optical_frame"/>
+    <origin xyz="0 0 0" rpy="-1.5707963267948966 0 -1.5707963267948966"/>
+  </joint>
   <gazebo reference="${prefix}camera_link">
-    <sensor name="rgbd_camera" type="rgbd_camera">
+    <sensor name="camera" type="rgbd_camera">
       <camera>
         <horizontal_fov>1.047</horizontal_fov>
@@ -17,5 +23,4 @@
           <far>8.0</far>
         </clip>
-        <frame_name>camera_rgb_optical_frame</frame_name>
       </camera>
       <always_on>1</always_on>
@@ -23,5 +28,5 @@
       <visualize>true</visualize>
       <topic>camera</topic>
-      <gz_frame_id>camera_link</gz_frame_id>
+      <frame_name>camera_rgb_optical_frame</frame_name>
     </sensor>
   </gazebo>

File: vicpinky_description/urdf/imu.xacro (robot description, xacro)
@@ -11,5 +11,4 @@
             <topic>imu</topic>
             <enable_metrics>true</enable_metrics>
-            <gz_frame_id>imu_link</gz_frame_id>
         </sensor>
     </gazebo>

File: vicpinky_description/urdf/robot_core.xacro (robot description, xacro)
@@ -258,16 +258,6 @@
       <origin xyz="0.07 0 0.56" rpy="0 0 0"/>
     </joint>
-    <link name="${prefix}camera_rgb_optical_frame"/>
-    <joint name="${prefix}camera_optical_joint" type="fixed">
-      <parent link="${prefix}camera_link"/>
-      <child link="${prefix}camera_rgb_optical_frame"/>
-      <origin xyz="0.035 0.015 0.008" rpy="0 0 0"/>
-      <pose>0 0 0 -1.57079632679 0 -1.57079632679</pose>
-      <axis>
-        <xyz>0 0 1</xyz>
-      </axis>
-    </joint>
     <!-- IMU -->
-    <joint name="imu_joint" type="fixed">
+    <joint name="${prefix}imu_joint" type="fixed">
         <origin xyz="0 0 0" rpy="0 0 0" />
         <parent link="base_link"/>

Commit message: [camera update]

File: vicpinky_description/urdf/camera.xacro (robot description, xacro)
@@ -1,13 +1,7 @@
 <?xml version="1.0"?>
 <robot xmlns:xacro="http://www.ros.org/wiki/xacro">
-  <xacro:arg name="namespace" default=""/>
-  <property name="prefix" value="$(arg namespace)"/>
-  <xacro:arg name="use_gazebo" default="true"/>
-  <link name="${prefix}camera_rgb_optical_frame"></link>
-  <joint name="${prefix}camera_optical_joint" type="fixed">
-    <parent link="${prefix}camera_link"/>
-    <child link="${prefix}camera_rgb_optical_frame"/>
-    <origin xyz="0 0 0" rpy="-1.5707963267948966 0 -1.5707963267948966"/>
-  </joint>
+    <xacro:arg name="namespace" default=""/>
+    <xacro:property name="prefix" value="$(arg namespace)"/>
+    <xacro:arg name="use_gazebo" default="true"/>
   <gazebo reference="${prefix}camera_link">
     <sensor name="camera" type="rgbd_camera">
@@ -23,4 +17,11 @@
           <far>8.0</far>
         </clip>
+        <depth_camera>
+          <clip>
+            <near>0.2</near>
+            <far>8.0</far>
+          </clip>
+        </depth_camera>
+        <optical_frame_id>${prefix}camera_rgb_optical_frame</optical_frame_id>
       </camera>
       <always_on>1</always_on>
@@ -28,5 +29,5 @@
       <visualize>true</visualize>
       <topic>camera</topic>
-      <frame_name>camera_rgb_optical_frame</frame_name>
+      <gz_frame_id>${prefix}camera_link</gz_frame_id>
     </sensor>
   </gazebo>

File: vicpinky_description/urdf/robot_core.xacro (robot description, xacro)
@@ -238,31 +238,59 @@
     <!-- Camera -->
     <link name="${prefix}camera_link">
-      <visual>
+    <visual>
         <geometry>
-          <mesh filename="package://vicpinky_description/meshes/visual/orbbec_astra_camera.dae"/>
+        <mesh filename="package://vicpinky_description/meshes/visual/orbbec_astra_camera.dae"/>
         </geometry>
-      </visual>
-      <collision>
+    </visual>
+    <collision>
         <geometry>
-          <box size="0.06 0.17 0.048"/>
+        <box size="0.06 0.17 0.048"/>
         </geometry>
-      </collision>
-      <inertial>
+    </collision>
+    <inertial>
         <mass value="0.22" />
         <inertia ixx="0.000513" ixy="0.0" ixz="0.0" iyy="0.000086" iyz="0.0" izz="0.0005"/>
-      </inertial>
+    </inertial>
     </link>
     <joint name="${prefix}camera_joint" type="fixed">
-      <parent link="${prefix}base_link"/>
-      <child link="${prefix}camera_link"/>
-      <origin xyz="0.07 0 0.56" rpy="0 0 0"/>
+        <parent link="${prefix}base_link"/>
+        <child link="${prefix}camera_link"/>
+        <origin xyz="0.07 0 0.56" rpy="0 0 0"/>
+    </joint>
+    <!-- RGB Frame -->
+    <link name="${prefix}camera_rgb_frame"/>
+    <joint name="${prefix}camera_rgb_joint" type="fixed">
+        <parent link="${prefix}camera_link"/>
+        <child link="${prefix}camera_rgb_frame"/>
+        <origin xyz="0.035 0.015 0.008" rpy="0 0 0"/>
+    </joint>
+    <!-- RGB Optical Frame -->
+    <link name="${prefix}camera_rgb_optical_frame"/>
+    <joint name="${prefix}camera_rgb_optical_joint" type="fixed">
+        <parent link="${prefix}camera_rgb_frame"/>
+        <child link="${prefix}camera_rgb_optical_frame"/>
+        <origin xyz="0 0 0" rpy="${-pi/2} 0 ${-pi/2}"/>
+    </joint>
+    <!-- Depth Frame -->
+    <link name="${prefix}camera_depth_frame"/>
+    <joint name="${prefix}camera_depth_joint" type="fixed">
+        <parent link="${prefix}camera_link"/>
+        <child link="${prefix}camera_depth_frame"/>
+        <origin xyz="0.035 0.015 0.008" rpy="0 0 0"/>
+    </joint>
+    <!-- Depth Optical Frame -->
+    <link name="${prefix}camera_depth_optical_frame"/>
+    <joint name="${prefix}camera_depth_optical_joint" type="fixed">
+        <parent link="${prefix}camera_depth_frame"/>
+        <child link="${prefix}camera_depth_optical_frame"/>
+        <origin xyz="0 0 0" rpy="${-pi/2} 0 ${-pi/2}"/>
     </joint>
     <!-- IMU -->
     <joint name="${prefix}imu_joint" type="fixed">
         <origin xyz="0 0 0" rpy="0 0 0" />
-        <parent link="base_link"/>
-        <child link="imu_link" />
-    </joint>
-    <link name="imu_link">
+        <parent link="${prefix}base_link"/>
+        <child link="${prefix}imu_link" />
+    </joint>
+    <link name="${prefix}imu_link">
     </link>
 </robot>
